File: production/sebik-ecad/LEDBoard/LEDBoard/LEDBoard.kicad_pcb (KiCad board)
At the start: 2 copper layers, 177.8 x 25.4 mm, 13 parts, among them J1 Conn_01x05_Male

Commit message: added project name
Parts:
- H1, H2, H3, H4: value MountingHole -> MountingHole_Pad
- moved H1 0.18 mm to (60.8, 81.2)
- moved H2 0.13 mm to (60.9, 96.4)
- moved H3 0.10 mm to (228.7, 96.5)
- moved H4 0.10 mm to (228.5, 81.3)
Connections:
- net Net-(J1-Pad1) renamed High Temp Yellow LED
- net Net-(J1-Pad2) renamed In Progress Yellow LED
- net Net-(J1-Pad3) renamed Low Temp Yellow LED
- net Net-(J1-Pad4) renamed High Pressure/Complete Yellow LED
