File: production/sebik-ecad/LEDBoard/LEDBoard/LEDBoard.kicad_sch (KiCad schematic)
At the start: 13 parts, among them J1 Conn_01x05_Male

Commit message: added project name
Parts:
- removed H1, H2, H3, H4: MountingHole, MountingHole:MountingHole_4.3mm_M4, symbol Mechanical:MountingHole
- added H1, H2, H3, H4: MountingHole_Pad, MountingHole:MountingHole_4.3mm_M4, symbol Mechanical:MountingHole_Pad
Connections:
- net GND: now also H1.1, H2.1, H3.1, H4.1
